File: HARDWARE/ZigZag/ZigZag.kicad_pcb (KiCad board)
At the start: 2 copper layers, 79.9 x 29.7 mm, 44 parts, among them SW1 SW_Push, T1 2N3904, U1 CH32V003J4M6(SOP8)

Commit message: Sync SCH and PCB
Parts:
- removed GND1 (x2): TESTPAD, OLIMEX_Other-FP:arc_90_0.5
- removed radiona: radiona, radiona:radiona
- added PAD2: TESTPAD, Custom:arc_90_0.5, F.Cu at (136.2, 108.4)
- moved R13 12.8 mm to (181.3, 115.9), turned to -135 degrees
- moved R12 8.19 mm to (180.2, 114.8), turned to -135 degrees
- moved TP2 1.11 mm to (177.9, 114.2)
Routing:
- net Net-(F_LED5-K): track 42.8 -> 31.2 mm, vias 1 -> 3
- net /PD1\SWIO\KBD_CLK: track 56.2 -> 67.7 mm, vias 1 -> 3
- net Net-(F_LED4-K): track 9.78 -> 19.9 mm
- net +5V: track 92.9 -> 100.6 mm, vias 0 -> 2
- net /PC2\T2CH2_1\Video_Out: track 30.9 -> 35.1 mm
- net GND: track 0.44 -> 2.60 mm, vias 15 -> 16
- net /PA2\KBD_DAT: track 52.0 -> 51.2 mm
- net /PD6\T2CH3_3\VSync: track 44.3 -> 43.5 mm
- net Net-(D1-K): track 26.6 -> 26.1 mm
