File: HARDWARE/ZigZag/ZigZag.kicad_sch (KiCad schematic)
At the start: 42 parts, among them SW1 SW_Push, T1 2N3904, U1 CH32V003J4M6(SOP8)

Commit message: uređena schema
Other:
- note added: "${project_creator} Liense: ${project_license} Year: ${project_year}"
- note added: "${project_name}"
- note added: "BOTTOM VIEW"
- note added: "TOP VIEW"
- company: Radiona Org -> ${project_creator}
- title: ZagZag -> ${project_name} ${project_version}
- moved on the sheet: AUD/UP1, BLU1, BT1, C1, D1, F_LED1, F_LED2, F_LED3, F_LED4, F_LED5, GND1, GRN1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

Commit message: Sync SCH and PCB
Parts:
- PAD2: renamed from GND1; footprint OLIMEX_Other-FP:arc_90_0.5 -> Custom:arc_90_0.5
Other:
- moved on the sheet: PAD2
Changed lines of the file:
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@@
 	)
 	(junction
-		(at 49.53 87.63)
-		(diameter 0)
-		(color 0 0 0 0)
-	)
-	(junction
 		(at 80.01 137.16)
 		(diameter 0)
@@
 	(wire
 		(pts
-			(xy 49.53 87.63) (xy 49.53 92.71)
-		)
-		(stroke
-			(width 0)
-			(type default)
-		)
-	)
-	(wire
-		(pts
 			(xy 80.01 137.16) (xy 80.01 142.24)
 		)
@@
 	(wire
 		(pts
+			(xy 38.1 92.71) (xy 38.1 88.9)
+		)
+		(stroke
+			(width 0)
+			(type default)
+		)
+	)
+	(wire
+		(pts
 			(xy 36.83 134.62) (xy 80.01 134.62)
 		)
@@
 	(wire
 		(pts
-			(xy 44.45 87.63) (xy 49.53 87.63)
-		)
-		(stroke
-			(width 0)
-			(type default)
-		)
-	)
-	(wire
-		(pts
 			(xy 146.05 40.64) (xy 184.15 40.64)
 		)
@@
 	(wire
 		(pts
-			(xy 49.53 62.23) (xy 49.53 87.63)
+			(xy 49.53 62.23) (xy 49.53 92.71)
 		)
 		(stroke
@@
 	(symbol
 		(lib_id "OLIMEX_OTHER:TESTPAD")
-		(at 41.91 87.63 180)
+		(at 38.1 86.36 90)
 		(unit 1)
 		(exclude_from_sim no)
@@
 		(on_board yes)
 		(dnp no)
-		(property "Reference" "GND1"
-			(at 36.83 87.63 0)
+		(property "Reference" "PAD2"
+			(at 38.1 81.28 0)
 			(effects
 				(font
@@
 		)
 		(property "Value" "TESTPAD"
-			(at 44.45 84.709 0)
+			(at 41.021 88.9 0)
 			(effects
 				(font
@@
 			)
 		)
-		(property "Footprint" "OLIMEX_Other-FP:arc_90_0.5"
-			(at 48.006 85.725 0)
+		(property "Footprint" "Custom:arc_90_0.5"
+			(at 40.005 92.456 0)
 			(effects
 				(font
@@
 		)
 		(property "Datasheet" ""
-			(at 41.91 87.63 90)
+			(at 38.1 86.36 90)
 			(effects
 				(font
@@
 		)
 		(property "Description" ""
-			(at 41.91 87.63 0)
+			(at 38.1 86.36 0)
 			(effects
 				(font
@@
 		)
 		(property "Fieldname 1" "Value 1"
-			(at 41.91 87.63 0)
+			(at 38.1 86.36 0)
 			(effects
 				(font
@@
 		)
 		(property "Fieldname2" "Value2"
-			(at 41.91 87.63 0)
+			(at 38.1 86.36 0)
 			(effects
 				(font
@@
 		)
 		(property "Fieldname3" "Value3"
-			(at 41.91 87.63 0)
+			(at 38.1 86.36 0)
 			(effects
 				(font
@@
 			(project "RVPC_Rev_B"
 				(path "/61827188-a485-403a-89e3-b210d5eae0ab"
-					(reference "GND1")
+					(reference "PAD2")
 					(unit 1)
 				)
@@
 					(unit 1)
 				)
+			)
+		)
+	)
+	(symbol
+		(lib_id "OLIMEX_Power:GND")
+		(at 38.1 92.71 0)
+		(unit 1)
+		(exclude_from_sim no)
+		(in_bom yes)
+		(on_board yes)
+		(dnp no)
+		(property "Reference" "#PWR021"
+			(at 38.1 99.06 0)
+			(effects
+				(font
+					(size 1.27 1.27)
+				)
+				(hide yes)
+			)
+		)
+		(property "Value" "GND"
+			(at 38.1 96.52 0)
+			(effects
+				(font
+					(size 1.27 1.27)
+				)
+			)
+		)
+		(property "Footprint" ""
+			(at 38.1 92.71 0)
+			(effects
+				(font
+					(size 1.524 1.524)
+				)
+			)
+		)
+		(property "Datasheet" ""
+			(at 38.1 92.71 0)
+			(effects
+				(font
+					(size 1.524 1.524)
+				)
+			)
+		)
+		(property "Description" ""
+			(at 38.1 92.71 0)
+			(effects
+				(font
+					(size 1.27 1.27)
+				)
+				(hide yes)
+			)
+		)
+		(pin "1"
+		)
+		(instances
+			(project "ZigZag"
+				(path "/61827188-a485-403a-89e3-b210d5eae0ab"
+					(reference "#PWR021")
+					(unit 1)
+				)
